File: Hardware/IN17BOARD.brd (EAGLE design)
At the start: 50 x 38 mm, 55 parts, among them IC1 IC_74141-DIP-16, J1 AVR_SPI_PRG_62X3_LOCK, Q1 MPSA42, Q2 MPSA92, Q3 MPSA42, Q4 MPSA92, Q5 MPSA42, Q6 MPSA92, Q7 MPSA42, Q8 MPSA92

Commit message: Add value and main sketch
Parts:
- C5: value (none) -> 0.1uf
- R17, R18, R19, R20: value (none) -> 220
Changed lines of the file:
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@@
 <element name="H1" library="holes" package="3,0" value="MOUNT-HOLE3.0" x="4.064" y="33.528"/>
 <element name="H2" library="holes" package="3,0" value="MOUNT-HOLE3.0" x="45.974" y="4.064"/>
-<element name="C5" library="SparkFun-Capacitors" package="0805" value="" x="32.766" y="36.068" smashed="yes" rot="MR0">
+<element name="C5" library="SparkFun-Capacitors" package="0805" value="0.1uf" x="32.766" y="36.068" smashed="yes" rot="MR0">
 <attribute name="NAME" x="34.3535" y="35.814" size="0.4064" layer="26" rot="MR90"/>
 <attribute name="VALUE" x="33.782" y="34.671" size="0.4064" layer="28" rot="MR0"/>
@@
 <element name="LED3" library="SparkFun-LED" package="LED-0603" value="" x="24.892" y="20.574"/>
 <element name="LED4" library="SparkFun-LED" package="LED-0603" value="" x="38.1" y="15.494" rot="R180"/>
-<element name="R17" library="SparkFun-Resistors" package="0603-RES" value="" x="11.684" y="12.446" rot="R270"/>
-<element name="R18" library="SparkFun-Resistors" package="0603-RES" value="" x="24.892" y="12.446" rot="R270"/>
-<element name="R19" library="SparkFun-Resistors" package="0603-RES" value="" x="24.892" y="23.622" rot="R90"/>
-<element name="R20" library="SparkFun-Resistors" package="0603-RES" value="" x="38.1" y="12.192" rot="R270"/>
+<element name="R17" library="SparkFun-Resistors" package="0603-RES" value="220" x="11.684" y="12.446" rot="R270"/>
+<element name="R18" library="SparkFun-Resistors" package="0603-RES" value="220" x="24.892" y="12.446" rot="R270"/>
+<element name="R19" library="SparkFun-Resistors" package="0603-RES" value="220" x="24.892" y="23.622" rot="R90"/>
+<element name="R20" library="SparkFun-Resistors" package="0603-RES" value="220" x="38.1" y="12.192" rot="R270"/>
 <element name="JP1" library="SparkFun-Connectors" package="1X09" value="M09" x="14.732" y="1.27" smashed="yes"/>
 <element name="H4" library="holes" package="3,0" value="MOUNT-HOLE3.0" x="45.974" y="33.528"/>
